Commit message: Trying SLAM and Navigation

File: toto2_description/models/toto2.xacro (robot description, xacro)
@@ -112,4 +112,12 @@
   <link name="camera_1">
   </link>
+  <link name="imu_link">
+  </link>
+  <joint name="imu_joint" type="fixed">
+      <parent link="base_link"/>
+      <child link="imu_link"/>
+      <origin xyz="0.0 0.0 0.17" rpy="0 0 0" />
+      <axis xyz="0.0 0.0 1.0" />
+    </joint>
   <joint name="camera_joint_1" type="fixed">
     <parent link="base_link"/>

Commit message: SLAM and Navigation completed

File: toto2_description/models/toto2.xacro (robot description, xacro)
@@ -6,4 +6,5 @@
   <xacro:include filename="$(find toto2_description)/urdf/toto.gazebo" /> -->
   <!-- BASE LINKS AND JOINTS OF ROBOT ARE IN THIS THESE ALLOW THE ROBOT TO NAVIGATE-->
+  <link name="base_footprint"/>
   <link name="base_link">
     <inertial>
@@ -114,10 +115,16 @@
   <link name="imu_link">
   </link>
+  <joint name="base" type="fixed">
+    <parent link="base_footprint"/>
+    <child link="base_link"/>
+    <origin xyz="0.0 0.0 0.1" rpy="0 0 0" />
+    <axis xyz="0.0 0.0 1.0" />
+  </joint>
   <joint name="imu_joint" type="fixed">
-      <parent link="base_link"/>
-      <child link="imu_link"/>
-      <origin xyz="0.0 0.0 0.17" rpy="0 0 0" />
-      <axis xyz="0.0 0.0 1.0" />
-    </joint>
+    <parent link="base_link"/>
+    <child link="imu_link"/>
+    <origin xyz="0.0 0.0 0.17" rpy="0 0 0" />
+    <axis xyz="0.0 0.0 1.0" />
+  </joint>
   <joint name="camera_joint_1" type="fixed">
     <parent link="base_link"/>
